Commit message: Changed the wheels urdf, not independetn joints but fixed to the chassis to avoid them lagging behind. Created a new topic, scan_filter, to modify the scan messages to make comaptible with SLAM toolbox (changed max_angle). SLAM is now working on the rover in real world.git add .git add .

File: src/leo_gazebo/description/leo_sim.xacro (robot description, xacro)
@@ -1,4 +1,5 @@
 <?xml version="1.0"?>
 <robot name="leo" xmlns:xacro="http://www.ros.org/wiki/xacro">
+    <!-- This version includes the wheels as cont. joints and they have axis and dynamics-->
     <!-- Base Link -->
     <link name="base_link">
@@ -47,8 +48,10 @@
         </inertial>
     </link>
-    <joint name="wheel_fl_chassis" type="fixed">
+    <joint name="wheel_fl_chassis" type="continuous">
         <origin xyz="0.1475 0.177 0.0" rpy="-1.5708 0 0" />
         <parent link="chassis" />
         <child link="wheel_fl" />
+        <axis xyz="0 0 1" />
+        <dynamics damping="0.7" friction="1.0" />
     </joint>
     <link name="wheel_fr">
@@ -69,8 +72,10 @@
         </inertial>
     </link>
-    <joint name="wheel_fr_chassis" type="fixed">
+    <joint name="wheel_fr_chassis" type="continuous">
         <origin xyz="0.1475 -0.177 0.0" rpy="-1.5708 0 0" />
         <parent link="chassis" />
         <child link="wheel_fr" />
+        <axis xyz="0 0 1" />
+        <dynamics damping="0.7" friction="1.0" />
     </joint>
     <link name="wheel_rl">
@@ -91,8 +96,10 @@
         </inertial>
     </link>
-    <joint name="wheel_rl_chassis" type="fixed">
+    <joint name="wheel_rl_chassis" type="continuous">
         <origin xyz="-0.1475 0.177 0.0" rpy="-1.5708 0 0" />
         <parent link="chassis" />
         <child link="wheel_rl" />
+        <axis xyz="0 0 1" />
+        <dynamics damping="0.7" friction="1.0" />
     </joint>
     <link name="wheel_rr">
@@ -113,8 +120,10 @@
         </inertial>
     </link>
-    <joint name="wheel_rr_chassis" type="fixed">
+    <joint name="wheel_rr_chassis" type="continuous">
         <origin xyz="-0.1475 -0.177 0.0" rpy="-1.5708 0 0" />
         <parent link="chassis" />
         <child link="wheel_rr" />
+        <axis xyz="0 0 1" />
+        <dynamics damping="0.7" friction="1.0" />
     </joint>
     <!-- Jetson Mount -->
@@ -241,5 +250,5 @@
         </sensor>
     </gazebo>
-    <!-- State publisher
+    <!-- State publisher -->
     <gazebo>
         <plugin name="gazebo_ros_joint_state_publisher"
@@ -252,4 +261,3 @@
         </plugin>
     </gazebo>
-    -->
 </robot>
